Commit message: modified table and mustard shapes

File: real_robots/data/kuka_gripper_description/urdf/table.urdf (robot description, URDF)
Before this commit: robot table, 1 links, 0 joints
Links:
- removed link table
- added link table_base, mass 0.0; collision mesh filename=package://kuka_gripper_description/meshes/table.obj; visual mesh filename=package://kuka_gripper_description/meshes/table.obj
- added link table_upper, mass 0.0; collision mesh filename=package://kuka_gripper_description/meshes/table_upper.obj; visual mesh filename=package://kuka_gripper_description/meshes/table_upper.obj
Joints:
- added joint upper: type fixed, parent table_base, child table_upper, origin xyz=0.0 0.0 0.0 rpy=0 0 0

Commit message: Fixed table width

File: real_robots/data/kuka_gripper_description/urdf/table.urdf (robot description, URDF)
Before this commit: robot table, 2 links, 1 joints
Links:
- link table_base: geometry collision mesh filename=package://kuka_gripper_description/meshes/table.obj scale=1.0 2.0 1.0; visual mesh filename=package://kuka_gripper_description/meshes/table.obj scale=1.0 2.0 1.0
- link table_upper: geometry collision mesh filename=package://kuka_gripper_description/meshes/table_upper.obj scale=1.0 2.0 1.0; visual mesh filename=package://kuka_gripper_description/meshes/table_upper.obj scale=1.0 2.0 1.0

Commit message: Rescaled table to 80cm width

File: real_robots/data/kuka_gripper_description/urdf/table.urdf (robot description, URDF)
Before this commit: robot table, 2 links, 1 joints
Links:
- link table_base: geometry collision mesh filename=package://kuka_gripper_description/meshes/table.obj scale=1.0 1.6 1.0; visual mesh filename=package://kuka_gripper_description/meshes/table.obj scale=1.0 1.6 1.0
- link table_upper: geometry collision mesh filename=package://kuka_gripper_description/meshes/table_upper.obj scale=1.0 1.6 1.0; visual mesh filename=package://kuka_gripper_description/meshes/table_upper.obj scale=1.0 1.6 1.0

Commit message: Improved table dimensions, effector speed, test_actions (WIP)

File: real_robots/data/kuka_gripper_description/urdf/table.urdf (robot description, URDF)
Before this commit: robot table, 2 links, 1 joints
Links:
- link table_base: geometry collision mesh filename=package://kuka_gripper_description/meshes/table.obj scale=1.1 2.0 1.0; visual mesh filename=package://kuka_gripper_description/meshes/table.obj scale=1.1 2.0 1.0
- link table_upper: geometry collision mesh filename=package://kuka_gripper_description/meshes/table_upper.obj scale=1.0 2.0 1.0; visual mesh filename=package://kuka_gripper_description/meshes/table_upper.obj scale=1.0 2.0 1.0
